Commit message: modified readme.md

File: kinova_description/urdf/kinova_common.xacro (robot description, xacro)
@@ -19,6 +19,5 @@
             <visual>
                 <geometry>
-                    <mesh
-                        filename="package://kinova_description/meshes/${link_mesh}.dae"/>
+                    <mesh filename="package://kinova_description/meshes/${link_mesh}.dae"/>
                 </geometry>
                 <material name="carbon_fiber">
