Commit message: modified 7dof model for gazebo 9

File: kinova_description/urdf/j2s6s300_standalone.xacro (robot description, xacro)
@@ -19,5 +19,5 @@
       <origin xyz="0 0 0" rpy="0 0 0" />
       <geometry>
-        <box size = "0 0 0"/>
+        <box size = "0.001 0.001 0.001"/>
       </geometry>
     <!--<material name="Black" /> -->
@@ -26,5 +26,5 @@
       <origin xyz="0 0 0" rpy="0 0 0" />
       <geometry>
-        <box size = "0 0 0"/>
+        <box size = "0.001 0.001 0.001"/>
       </geometry>
     </collision>

File: kinova_description/urdf/j2s7s300.xacro (robot description, xacro)
@@ -60,5 +60,5 @@
     <property name="joint_2_upper_limit" value="${313/180*J_PI}" />
     <property name="joint_3" value="joint_3" />
-    <property name="joint_3_type" value="continuous" />
+    <property name="joint_3_type" value="revolute" />
     <property name="joint_3_axis_xyz" value="0 0 1" />
     <property name="joint_3_origin_xyz" value="0 -0.205 0" />

File: kinova_description/urdf/j2s7s300_standalone.xacro (robot description, xacro)
@@ -19,5 +19,5 @@
       <origin xyz="0 0 0" rpy="0 0 0" />
       <geometry>
-        <box size = "0 0 0"/>
+        <box size = "0.001 0.001 0.001"/>
       </geometry>
     <!--<material name="Black" /> -->
@@ -26,5 +26,5 @@
       <origin xyz="0 0 0" rpy="0 0 0" />
       <geometry>
-        <box size = "0 0 0"/>
+        <box size = "0.001 0.001 0.001"/>
       </geometry>
     </collision>

File: kinova_description/urdf/kinova_common.xacro (robot description, xacro)
@@ -56,5 +56,6 @@
         <type>transmission_interface/SimpleTransmission</type>
         <joint name="${joint_name}">
-          <hardwareInterface>EffortJointInterface</hardwareInterface>
+          <!-- hardwareInterface>EffortJointInterface</hardwareInterface-->
+          <hardwareInterface>hardware_interface/EffortJointInterface</hardwareInterface>
         </joint>
         <actuator name="${joint_name}_actuator">
@@ -100,5 +101,6 @@
 					<type>transmission_interface/SimpleTransmission</type>
 					<joint name="${prefix}joint_finger_${finger_number}">
-					  <hardwareInterface>EffortJointInterface</hardwareInterface>
+					  <!--hardwareInterface>EffortJointInterface</hardwareInterface-->
+                      <hardwareInterface>hardware_interface/EffortJointInterface</hardwareInterface>
 					</joint>
 					<actuator name="${prefix}joint_finger_${finger_number}_actuator">
